Commit message: inne wartosci kątów + wykres

File: lab2/urdf/fixed.urdf (robot description, URDF)
Before this commit: robot fixed_robot, 4 links, 3 joints
Joints:
- joint base to link_1: origin xyz=0 0 0.1 rpy=0 0 1 -> xyz=0 0 0.1 rpy=0 0 0.78539
- joint link_1 to link_2: origin xyz=0 0 0.2 rpy=-1.57 -0.6 0 -> xyz=0 0 0.2 rpy=-1.57 -0.523 0
- joint link_2 to link_3: origin xyz=0.4 0 0 rpy=0 0 0.5 -> xyz=0.4 0 0 rpy=0 0 1.0471

File: lab2/urdf/movable.urdf (robot description, URDF)
Before this commit: robot fixed_robot, 4 links, 3 joints
Joints:
- joint base to link_1: origin xyz=0 0 0.1 rpy=0 0 1 -> xyz=0 0 0.1 rpy=0 0 0.78539
- joint link_1 to link_2: origin xyz=0 0 0.2 rpy=-1.57 -0.6 0 -> xyz=0 0 0.2 rpy=-1.57 -0.523 0
- joint link_2 to link_3: origin xyz=0.4 0 0 rpy=0 0 0.5 -> xyz=0.4 0 0 rpy=0 0 1.0471
