Commit message: Poprawka kolejna

File: lab2/urdf/fixed (kopia).urdf (robot description, URDF)
Before this commit: robot movable_robot, 4 links, 3 joints
Joints:
- joint base to link_1: axis 0 0 1 -> (none); origin xyz=0 0 0 rpy=0 0 0.78539 -> xyz=0 0 0.1 rpy=0 0 0.78539; type continuous -> fixed
- joint link_1 to link_2: axis 0 0 1 -> (none); type continuous -> fixed
- joint link_2 to link_3: axis 0 0 1 -> (none); type continuous -> fixed

File: lab2/urdf/fixed.urdf (robot description, URDF)
Before this commit: robot fixed_robot, 4 links, 3 joints
Joints:
- joint base to link_1: origin xyz=0 0 0.1 rpy=0 0 0.78539 -> xyz=0 0 0 rpy=0 0 0.78539
