Commit message: zrobione nonkdl

File: lab3/urdf/movable.urdf (robot description, URDF)
Before this commit: robot movable_robot, 4 links, 3 joints
Joints:
- joint link_1 to link_2: limit (none) -> lower=-0.7853 upper=0.7853 effort=1000.0 velocity=0.5; origin xyz=0 0 0.2 rpy=-1.57 0 0 -> xyz=0 0 0.2 rpy=-1.57 -0.7853 0; type continuous -> revolute
- joint link_2 to link_3: limit (none) -> lower=-0.7853 upper=0.7853 effort=1000.0 velocity=0.5; origin xyz=0.4 0 0 rpy=0 0 0 -> xyz=0.4 0 0 rpy=0 0 0.7853; type continuous -> revolute

Commit message: test

File: lab3/urdf/movable.urdf (robot description, URDF)
Before this commit: robot movable_robot, 4 links, 3 joints
Joints:
- joint link_1 to link_2: origin xyz=0 0 0.2 rpy=-1.57 -0.7853 0 -> xyz=0 0 0.2 rpy=-1.57 0 0
- joint link_2 to link_3: origin xyz=0.4 0 0 rpy=0 0 0.7853 -> xyz=0.4 0 0 rpy=0 0 0
